File: CalmaAcc_hw/CalmaAcc.sch (KiCad schematic (older format))
At the start: 1 part

Commit message: sch 5%
Parts:
- added C? (x2): 0.1u, CAP_0603, symbol C
- added C?: 4.7u, CAP_0603, symbol C
- added C?: 10n, CAP_0603, symbol C
- added C?: 1u, CAP_0603, symbol C
Connections:
- net labels added: +3.3V, GND
- wire segments 0 -> 15
- no-connect marks 0 -> 3
Changed lines of the file:
@@
 LIBS:st_kl
 LIBS:Transistors_kl
+LIBS:CalmaAcc-cache
 EELAYER 25 0
 EELAYER END
@@
 	1    0    0    -1
 $EndComp
+$Comp
+L C C?
+U 1 1 56470FC3
+P 3950 3700
+F 0 "C?" H 3850 3600 50  0000 L CNN
+F 1 "0.1u" H 3850 3800 50  0000 L CNN
+F 2 "CAP_0603" V 4050 3550 28  0000 C BNN
+F 3 "" H 3950 3700 60  0000 C CNN
+	1    3950 3700
+	1    0    0    -1
+$EndComp
+$Comp
+L C C?
+U 1 1 5647102D
+P 3650 3700
+F 0 "C?" H 3550 3600 50  0000 L CNN
+F 1 "0.1u" H 3550 3800 50  0000 L CNN
+F 2 "CAP_0603" V 3750 3550 28  0000 C BNN
+F 3 "" H 3650 3700 60  0000 C CNN
+	1    3650 3700
+	1    0    0    -1
+$EndComp
+$Comp
+L C C?
+U 1 1 5647104C
+P 3350 3700
+F 0 "C?" H 3250 3600 50  0000 L CNN
+F 1 "4.7u" H 3250 3800 50  0000 L CNN
+F 2 "CAP_0603" V 3450 3550 28  0000 C BNN
+F 3 "" H 3350 3700 60  0000 C CNN
+	1    3350 3700
+	1    0    0    -1
+$EndComp
+$Comp
+L C C?
+U 1 1 56471098
+P 3050 3700
+F 0 "C?" H 2950 3600 50  0000 L CNN
+F 1 "10n" H 2950 3800 50  0000 L CNN
+F 2 "CAP_0603" V 3150 3550 28  0000 C BNN
+F 3 "" H 3050 3700 60  0000 C CNN
+	1    3050 3700
+	1    0    0    -1
+$EndComp
+$Comp
+L C C?
+U 1 1 564710BB
+P 2750 3700
+F 0 "C?" H 2650 3600 50  0000 L CNN
+F 1 "1u" H 2650 3800 50  0000 L CNN
+F 2 "CAP_0603" V 2850 3550 28  0000 C BNN
+F 3 "" H 2750 3700 60  0000 C CNN
+	1    2750 3700
+	1    0    0    -1
+$EndComp
+Wire Wire Line
+	3850 3300 4250 3300
+Wire Wire Line
+	3950 3300 3950 3500
+Wire Wire Line
+	3250 3200 4250 3200
+Wire Wire Line
+	3350 3200 3350 3500
+Wire Wire Line
+	3650 3500 3650 3200
+Connection ~ 3650 3200
+Wire Wire Line
+	2650 3100 4250 3100
+Wire Wire Line
+	2750 3100 2750 3500
+Wire Wire Line
+	3050 3500 3050 3100
+Connection ~ 3050 3100
+$Comp
+L GND #PWR?
+U 1 1 56471133
+P 3950 4100
+F 0 "#PWR?" H 4040 4080 30  0001 C CNN
+F 1 "GND" H 3950 4020 30  0001 C CNN
+F 2 "" H 3950 4100 60  0000 C CNN
+F 3 "" H 3950 4100 60  0000 C CNN
+	1    3950 4100
+	1    0    0    -1
+$EndComp
+$Comp
+L GND #PWR?
+U 1 1 56471153
+P 3650 4100
+F 0 "#PWR?" H 3740 4080 30  0001 C CNN
+F 1 "GND" H 3650 4020 30  0001 C CNN
+F 2 "" H 3650 4100 60  0000 C CNN
+F 3 "" H 3650 4100 60  0000 C CNN
+	1    3650 4100
+	1    0    0    -1
+$EndComp
+$Comp
+L GND #PWR?
+U 1 1 56471173
+P 3350 4100
+F 0 "#PWR?" H 3440 4080 30  0001 C CNN
+F 1 "GND" H 3350 4020 30  0001 C CNN
+F 2 "" H 3350 4100 60  0000 C CNN
+F 3 "" H 3350 4100 60  0000 C CNN
+	1    3350 4100
+	1    0    0    -1
+$EndComp
+$Comp
+L GND #PWR?
+U 1 1 56471193
+P 3050 4100
+F 0 "#PWR?" H 3140 4080 30  0001 C CNN
+F 1 "GND" H 3050 4020 30  0001 C CNN
+F 2 "" H 3050 4100 60  0000 C CNN
+F 3 "" H 3050 4100 60  0000 C CNN
+	1    3050 4100
+	1    0    0    -1
+$EndComp
+$Comp
+L GND #PWR?
+U 1 1 564711B3
+P 2750 4100
+F 0 "#PWR?" H 2840 4080 30  0001 C CNN
+F 1 "GND" H 2750 4020 30  0001 C CNN
+F 2 "" H 2750 4100 60  0000 C CNN
+F 3 "" H 2750 4100 60  0000 C CNN
+	1    2750 4100
+	1    0    0    -1
+$EndComp
+Wire Wire Line
+	3950 3900 3950 4100
+Wire Wire Line
+	3650 3900 3650 4100
+Wire Wire Line
+	3350 3900 3350 4100
+Wire Wire Line
+	3050 3900 3050 4100
+Wire Wire Line
+	2750 3900 2750 4100
+$Comp
+L +3.3V #PWR?
+U 1 1 56471423
+P 3850 3300
+F 0 "#PWR?" H 3850 3260 30  0001 C CNN
+F 1 "+3.3V" H 3930 3330 30  0000 C CNN
+F 2 "" H 3850 3300 60  0000 C CNN
+F 3 "" H 3850 3300 60  0000 C CNN
+	1    3850 3300
+	-1   0    0    1
+$EndComp
+$Comp
+L +3.3V #PWR?
+U 1 1 56471443
+P 3250 3200
+F 0 "#PWR?" H 3250 3160 30  0001 C CNN
+F 1 "+3.3V" H 3330 3230 30  0000 C CNN
+F 2 "" H 3250 3200 60  0000 C CNN
+F 3 "" H 3250 3200 60  0000 C CNN
+	1    3250 3200
+	-1   0    0    1
+$EndComp
+$Comp
+L +3.3V #PWR?
+U 1 1 5647147F
+P 2650 3100
+F 0 "#PWR?" H 2650 3060 30  0001 C CNN
+F 1 "+3.3V" H 2730 3130 30  0000 C CNN
+F 2 "" H 2650 3100 60  0000 C CNN
+F 3 "" H 2650 3100 60  0000 C CNN
+	1    2650 3100
+	-1   0    0    1
+$EndComp
+Connection ~ 3950 3300
+Connection ~ 3350 3200
+Connection ~ 2750 3100
+$Comp
+L GND #PWR?
+U 1 1 564714EA
+P 7450 3500
+F 0 "#PWR?" H 7540 3480 30  0001 C CNN
+F 1 "GND" H 7450 3420 30  0001 C CNN
+F 2 "" H 7450 3500 60  0000 C CNN
+F 3 "" H 7450 3500 60  0000 C CNN
+	1    7450 3500
+	1    0    0    -1
+$EndComp
+Wire Wire Line
+	7350 3300 7450 3300
+Wire Wire Line
+	7450 3300 7450 3500
+NoConn ~ 4250 3000
+NoConn ~ 4250 2800
+NoConn ~ 4250 2700
 $EndSCHEMATC

Commit message: + acc
Parts:
- added B?: BAT, symbol BAT
- added C? (x2): 47u, CAP_0805, symbol C
- added C?: 4.7u, CAP_0603, symbol C
- added C? (x2): 0.1u, CAP_0603, symbol C
- added D?: BAT54WS, symbol D_Shottky
- added DD?: MMA8452Q, symbol MMA8452Q
- added M?: MOTOR_PAD, symbol MOTOR_PAD
- added Q?: MMBT2222, symbol NPN
- added R?: 1k, RES_0603, symbol R
- added R? (x2): 4k7, RES_0603, symbol R
- added XL?: CONN_2, symbol CONN_2
Connections:
- net labels added: +BATT, ACC_INT1, I2C_SCL, I2C_SDA, Vibro
- net labels removed: +3.3V
- wire segments 15 -> 59
- no-connect marks 3 -> 4
Other:
- moved on the sheet: C?, DD?

Commit message: scheme done?
Parts:
- added D? (x3): LED, symbol LED
- added R? (x3): 51R, RES_0603, symbol R
Connections:
- net GND: now also D?.C, D?.C, D?.C
- net at DD?.12 (MISO1/T3C1/T16C1/PA6): now also R?.2
- net at DD?.13 (MOSI1/T3C2/T14C1/T1C1N/T17C1/PA7): now also R?.2
- net at DD?.14 (PB0/T3C3/T1C2N): now also R?.1
- new net: D?.A, R?.2
- new net: D?.A, R?.1 (x2)
Other:
- moved on the sheet: B?, C?, D?, DD?, M?, Q?, R?, XL?

Commit message: scheme update
Parts:
- removed M?: MOTOR_PAD, symbol MOTOR_PAD
Other:
- moved on the sheet: C?, D?, Q?, R?, XL?
Changed lines of the file:
@@
 	-1   0    0    1
-$EndComp
-$Comp
-L MOTOR_PAD M?
-U 1 1 564889FE
-P 12800 6450
-F 0 "M?" H 12550 6700 60  0000 C CNN
-F 1 "MOTOR_PAD" H 12950 6700 60  0000 C CNN
-F 2 "" H 12800 6450 60  0000 C CNN
-F 3 "" H 12800 6450 60  0000 C CNN
-	1    12800 6450
-	0    -1   -1   0
-$EndComp
-$Comp
-L GND #PWR?
-U 1 1 56488A75
-P 13350 6600
-F 0 "#PWR?" H 13440 6580 30  0001 C CNN
-F 1 "GND" H 13350 6520 30  0001 C CNN
-F 2 "" H 13350 6600 60  0000 C CNN
-F 3 "" H 13350 6600 60  0000 C CNN
-	1    13350 6600
-	1    0    0    -1
 $EndComp
 Wire Wire Line
@@
 Wire Wire Line
 	8350 8450 8800 8450
-Wire Wire Line
-	13200 6450 13350 6450
-Wire Wire Line
-	13350 6450 13350 6600
 $Comp
 L C C?
 U 1 1 56488B03
-P 12200 6200
-F 0 "C?" H 12100 6100 50  0000 L CNN
-F 1 "47u" H 12100 6300 50  0000 L CNN
-F 2 "CAP_0805" V 12300 6050 28  0000 C BNN
-F 3 "" H 12200 6200 60  0000 C CNN
-	1    12200 6200
+P 13350 6200
+F 0 "C?" H 13250 6100 50  0000 L CNN
+F 1 "47u" H 13250 6300 50  0000 L CNN
+F 2 "CAP_0805" V 13450 6050 28  0000 C BNN
+F 3 "" H 13350 6200 60  0000 C CNN
+	1    13350 6200
 	1    0    0    -1
 $EndComp
@@
 L C C?
 U 1 1 56488B5E
-P 11900 6200
-F 0 "C?" H 11800 6100 50  0000 L CNN
-F 1 "47u" H 11800 6300 50  0000 L CNN
-F 2 "CAP_0805" V 12000 6050 28  0000 C BNN
-F 3 "" H 11900 6200 60  0000 C CNN
-	1    11900 6200
+P 13050 6200
+F 0 "C?" H 12950 6100 50  0000 L CNN
+F 1 "47u" H 12950 6300 50  0000 L CNN
+F 2 "CAP_0805" V 13150 6050 28  0000 C BNN
+F 3 "" H 13050 6200 60  0000 C CNN
+	1    13050 6200
 	1    0    0    -1
 $EndComp
@@
 L +BATT #PWR?
 U 1 1 56488C25
-P 11500 5950
-F 0 "#PWR?" H 11500 5910 30  0001 C CNN
-F 1 "+BATT" H 11580 5980 30  0000 C CNN
-F 2 "" H 11500 5950 60  0000 C CNN
-F 3 "" H 11500 5950 60  0000 C CNN
-	1    11500 5950
+P 12650 5950
+F 0 "#PWR?" H 12650 5910 30  0001 C CNN
+F 1 "+BATT" H 12730 5980 30  0000 C CNN
+F 2 "" H 12650 5950 60  0000 C CNN
+F 3 "" H 12650 5950 60  0000 C CNN
+	1    12650 5950
 	-1   0    0    1
 $EndComp
@@
 L D_Shottky D?
 U 1 1 56488C75
-P 13750 6500
-F 0 "D?" H 13750 6600 40  0000 C CNN
-F 1 "BAT54WS" H 13750 6400 40  0000 C CNN
-F 2 "" H 13750 6500 60  0000 C CNN
-F 3 "" H 13750 6500 60  0000 C CNN
-	1    13750 6500
+P 13750 6200
+F 0 "D?" H 13750 6300 40  0000 C CNN
+F 1 "BAT54WS" H 13750 6100 40  0000 C CNN
+F 2 "" H 13750 6200 60  0000 C CNN
+F 3 "" H 13750 6200 60  0000 C CNN
+	1    13750 6200
 	0    -1   -1   0
 $EndComp
@@
 L CONN_2 XL?
 U 1 1 56488D61
-P 14450 6450
-F 0 "XL?" V 14400 6450 40  0000 C CNN
-F 1 "CONN_2" V 14500 6450 40  0000 C CNN
-F 2 "" H 14450 6450 60  0000 C CNN
-F 3 "" H 14450 6450 60  0000 C CNN
-	1    14450 6450
-	1    0    0    -1
-$EndComp
-Wire Wire Line
-	12800 6000 12800 5950
-Wire Wire Line
-	11500 5950 14250 5950
-Wire Wire Line
-	11900 6000 11900 5950
-Connection ~ 11900 5950
-Wire Wire Line
-	12200 6000 12200 5950
-Connection ~ 12200 5950
-Wire Wire Line
-	13750 5950 13750 6300
-Connection ~ 12800 5950
-Wire Wire Line
-	14250 5950 14250 6350
-Connection ~ 13750 5950
+P 14250 6650
+F 0 "XL?" V 14200 6650 40  0000 C CNN
+F 1 "CONN_2" V 14300 6650 40  0000 C CNN
+F 2 "" H 14250 6650 60  0000 C CNN
+F 3 "" H 14250 6650 60  0000 C CNN
+	1    14250 6650
+	1    0    0    -1
+$EndComp
+Wire Wire Line
+	13050 6000 13050 5950
+Connection ~ 13050 5950
+Wire Wire Line
+	13350 5950 13350 6000
 $Comp
 L GND #PWR?
 U 1 1 56488E9B
-P 12200 6550
-F 0 "#PWR?" H 12290 6530 30  0001 C CNN
-F 1 "GND" H 12200 6470 30  0001 C CNN
-F 2 "" H 12200 6550 60  0000 C CNN
-F 3 "" H 12200 6550 60  0000 C CNN
-	1    12200 6550
+P 13350 6550
+F 0 "#PWR?" H 13440 6530 30  0001 C CNN
+F 1 "GND" H 13350 6470 30  0001 C CNN
+F 2 "" H 13350 6550 60  0000 C CNN
+F 3 "" H 13350 6550 60  0000 C CNN
+	1    13350 6550
 	1    0    0    -1
 $EndComp
@@
 L GND #PWR?
 U 1 1 56488EC7
-P 11900 6550
-F 0 "#PWR?" H 11990 6530 30  0001 C CNN
-F 1 "GND" H 11900 6470 30  0001 C CNN
-F 2 "" H 11900 6550 60  0000 C CNN
-F 3 "" H 11900 6550 60  0000 C CNN
-	1    11900 6550
-	1    0    0    -1
-$EndComp
-Wire Wire Line
-	12200 6400 12200 6550
-Wire Wire Line
-	11900 6400 11900 6550
+P 13050 6550
+F 0 "#PWR?" H 13140 6530 30  0001 C CNN
+F 1 "GND" H 13050 6470 30  0001 C CNN
+F 2 "" H 13050 6550 60  0000 C CNN
+F 3 "" H 13050 6550 60  0000 C CNN
+	1    13050 6550
+	1    0    0    -1
+$EndComp
+Wire Wire Line
+	13350 6400 13350 6550
+Wire Wire Line
+	13050 6400 13050 6550
 $Comp
 L NPN Q?
 U 1 1 56488F54
-P 12750 7350
-F 0 "Q?" H 12950 7400 60  0000 C CNN
-F 1 "MMBT2222" H 13100 7300 60  0000 C CNN
-F 2 "" H 12750 7350 60  0000 C CNN
-F 3 "" H 12750 7350 60  0000 C CNN
-	1    12750 7350
+P 13700 7050
+F 0 "Q?" H 13900 7100 60  0000 C CNN
+F 1 "MMBT2222" H 14050 7000 60  0000 C CNN
+F 2 "" H 13700 7050 60  0000 C CNN
+F 3 "" H 13700 7050 60  0000 C CNN
+	1    13700 7050
 	1    0    0    -1
 $EndComp
@@
 L GND #PWR?
 U 1 1 56489007
-P 12800 7750
-F 0 "#PWR?" H 12890 7730 30  0001 C CNN
-F 1 "GND" H 12800 7670 30  0001 C CNN
-F 2 "" H 12800 7750 60  0000 C CNN
-F 3 "" H 12800 7750 60  0000 C CNN
-	1    12800 7750
-	1    0    0    -1
-$EndComp
-Wire Wire Line
-	12800 7550 12800 7750
-Wire Wire Line
-	12800 6900 12800 7150
-Wire Wire Line
-	13750 6700 13750 7000
-Wire Wire Line
-	12800 7000 14250 7000
-Connection ~ 12800 7000
-Wire Wire Line
-	14250 7000 14250 6550
-Connection ~ 13750 7000
+P 13750 7450
+F 0 "#PWR?" H 13840 7430 30  0001 C CNN
+F 1 "GND" H 13750 7370 30  0001 C CNN
+F 2 "" H 13750 7450 60  0000 C CNN
+F 3 "" H 13750 7450 60  0000 C CNN
+	1    13750 7450
+	1    0    0    -1
+$EndComp
+Wire Wire Line
+	13750 7250 13750 7450
 $Comp
 L R R?
 U 1 1 5648910B
-P 12050 7350
-F 0 "R?" V 12130 7200 50  0000 C CNN
-F 1 "1k" V 12050 7350 50  0000 C CNN
-F 2 "RES_0603" V 12130 7450 28  0000 C CNN
-F 3 "" H 12050 7350 60  0000 C CNN
-	1    12050 7350
-	0    1    1    0
-$EndComp
-Wire Wire Line
-	12550 7350 12300 7350
-Wire Wire Line
-	11800 7350 11300 7350
-Text Label 11300 7350 0    60   ~ 0
+P 13000 7050
+F 0 "R?" V 13080 6900 50  0000 C CNN
+F 1 "1k" V 13000 7050 50  0000 C CNN
+F 2 "RES_0603" V 13080 7150 28  0000 C CNN
+F 3 "" H 13000 7050 60  0000 C CNN
+	1    13000 7050
+	0    1    1    0
+$EndComp
+Wire Wire Line
+	13500 7050 13250 7050
+Text Label 12450 7050 0    60   ~ 0
 Vibro
 Text Label 10450 2250 2    60   ~ 0
@@
 Wire Wire Line
 	6100 1850 6300 1850
+Connection ~ 13350 5950
+Wire Wire Line
+	13750 5950 13750 6000
+Connection ~ 13750 5950
+Wire Wire Line
+	12750 7050 12450 7050
+Wire Wire Line
+	12650 5950 14050 5950
+Wire Wire Line
+	14050 5950 14050 6550
+Wire Wire Line
+	14050 6750 13750 6750
+Wire Wire Line
+	13750 6400 13750 6850
+Connection ~ 13750 6750
 $EndSCHEMATC

Commit message: scheme update
Parts:
- added XL?: CONN_3, symbol CONN_3
- added XL?: ST_SWD, symbol ST_SWD
Connections:
- net +BATT: now also XL?.1 (Vdd)
- net GND: now also XL?.1 (P1), XL?.3 (GND)
- net SWDIO: now reaches DD?.21 (SWDIO/PA13)
- net SWDIO: now also XL?.4 (SWDIO)
- net SWCLK: now reaches DD?.22 (SWCLK/PA14)
- net SWCLK: now also XL?.2 (SWCLK)
- net UART_TX: now reaches DD?.8 (ADC2/WKUP4/T2C3/TX2/PA2)
- net UART_TX: now also XL?.2 (PM)
- net UART_RX: now reaches DD?.9 (ADC3/T2C4/RX2/PA3)
- net UART_RX: now also XL?.3
- no-connect marks 4 -> 14
Other:
- note added: "Accelerometer"
- note added: "Debug port"
- note added: "Programming"
- note added: "Vibro"
- moved on the sheet: B?, C?, D?, DD?, Q?, R?, XL?

Commit message: + net
Parts:
- C1, C2, C3, C4, C5, C6, C7, C8: renamed from C?; footprint CAP_0603 -> Capacitors:CAP_0402
- C10, C9: renamed from C?; footprint CAP_0805 -> Capacitors:CAP_0805
- D1, D3, D4: renamed from D?; footprint (none) -> LEDs:LED_0603
- D2: renamed from D?; footprint (none) -> Diodes:SOD323
- DD1: renamed from DD?; footprint (none) -> QFN_DFN:QFN16_5_3
- Q1: renamed from Q?; footprint (none) -> SOT:SOT23-3
- R1, R2, R3, R4, R5, R6: renamed from R?; footprint RES_0603 -> Resistors:RES_0402
- XL1: renamed from XL?; footprint (none) -> Connectors:PLS-4
- XL2: renamed from XL?; footprint (none) -> Connectors:PLS-3
- XL3: renamed from XL?; footprint (none) -> Connectors:PLS-2
- gave numbers to parts that had none: 2
Connections:
- no-connect marks 14 -> 15

Commit message: +pcb and toporrrrr
Parts:
- B1: footprint (none) -> Batteries_kl:BAT_CH7410
- DD2: footprint (none) -> QFN_DFN:UFQFPN28
- renumbered XL2 to XL4
Connections:
- net Vibro_out: now reaches D2.A, Q1.3 (C), XL3.2 (PM)
Changed lines of the file:
@@
 F 0 "DD2" H 8850 4800 60  0000 C CNN
 F 1 "STM32F042G4" H 9400 4800 60  0000 C CNN
-F 2 "" H 9400 3050 60  0001 C CNN
+F 2 "QFN_DFN:UFQFPN28" H 9400 3050 60  0001 C CNN
 F 3 "" H 9400 3050 60  0000 C CNN
 	1    9350 3350
@@
 F 0 "B1" H 2250 5750 60  0000 C CNN
 F 1 "BAT" H 1850 5750 60  0000 C CNN
-F 2 "" H 2100 5550 60  0001 C CNN
+F 2 "Batteries_kl:BAT_CH7410" H 2100 5550 60  0001 C CNN
 F 3 "" H 2100 5550 60  0000 C CNN
 	1    2100 5550
@@
 Connection ~ 11750 8350
 $Comp
-L CONN_3 XL2
+L CONN_3 XL4
 U 1 1 5648B6D3
 P 2050 3900
-F 0 "XL2" V 2000 3900 40  0000 C CNN
+F 0 "XL4" V 2000 3900 40  0000 C CNN
 F 1 "CONN_3" V 2100 3900 40  0000 C CNN
 F 2 "Connectors:PLS-3" H 2050 3900 60  0001 C CNN
@@
 NoConn ~ 10900 3300
 NoConn ~ 17600 2100
+Text Label 11750 8300 1    60   ~ 0
+Vibro_out
 $EndSCHEMATC

Commit message: +STM32F042F6
Parts:
- removed C8: 0.1u, Capacitors:CAP_0402, symbol C
- removed DD2: STM32F042G4, QFN_DFN:UFQFPN28, symbol STM32F042G4
- added DD?: STM32F042F6P6, symbol STM32F042F6P6
Connections:
- net +BATT: now also DD?.16 (VDD), DD?.5 (VDDA)
- net ACC_INT1: now also DD?.6 (ADC0/WKUP1/T2C1/PA0)
- net GND: now also DD?.15 (VSS)
- net I2C_SCL: now also DD?.3 (PF1/OSCOUT/SCL1)
- net I2C_SDA: now also DD?.2 (PF0/OSCIN/SDA1)
- net SWCLK: now also DD?.20 (SWCLK/PA14)
- net SWDIO: now also DD?.19 (SWDIO/PA13)
- net UART_RX: now also DD?.9 (ADC3/T2C4/RX2/PA3)
- net UART_TX: now also DD?.8 (ADC2/WKUP4/T2C3/TX2/PA2)
- net Vibro: now also DD?.10 (T14C1/PA4)
- net at R5.2: now also DD?.12 (MISO1/T3C1/T16C1/PA6)
- net at R6.2: now also DD?.13 (MOSI1/T3C2/T14C1/T1C1N/T17C1/PA7)
- net at R3.1: now also DD?.14 (PB1/T3C4/T14C1/T1C3N)
- no-connect marks 15 -> 8
Other:
- moved on the sheet: C4, C5, C6, C7, D1, D3, D4, R3, R5, R6
