File: CalmaAcc_hw/CalmaAcc.sch (KiCad schematic (older format))
At the start: 26 parts, among them Q1 MMBT2222

Commit message: + TSSOP20
Parts:
- DD2: renamed from DD?; footprint (none) -> SO_DIL_TSSOP:TSSOP20
- R3, R5, R6: value 51R -> 100R
Changed lines of the file:
@@
 $EndComp
 $Comp
-L GND #PWR02
+L GND #PWR01
 U 1 1 56471153
 P 6400 4200
-F 0 "#PWR02" H 6490 4180 30  0001 C CNN
+F 0 "#PWR01" H 6490 4180 30  0001 C CNN
 F 1 "GND" H 6400 4120 30  0001 C CNN
 F 2 "" H 6400 4200 60  0000 C CNN
@@
 $EndComp
 $Comp
-L GND #PWR03
+L GND #PWR02
 U 1 1 56471173
 P 6100 4200
-F 0 "#PWR03" H 6190 4180 30  0001 C CNN
+F 0 "#PWR02" H 6190 4180 30  0001 C CNN
 F 1 "GND" H 6100 4120 30  0001 C CNN
 F 2 "" H 6100 4200 60  0000 C CNN
@@
 $EndComp
 $Comp
-L GND #PWR04
+L GND #PWR03
 U 1 1 56471193
 P 5800 4200
-F 0 "#PWR04" H 5890 4180 30  0001 C CNN
+F 0 "#PWR03" H 5890 4180 30  0001 C CNN
 F 1 "GND" H 5800 4120 30  0001 C CNN
 F 2 "" H 5800 4200 60  0000 C CNN
@@
 $EndComp
 $Comp
-L GND #PWR05
+L GND #PWR04
 U 1 1 564711B3
 P 5500 4200
-F 0 "#PWR05" H 5590 4180 30  0001 C CNN
+F 0 "#PWR04" H 5590 4180 30  0001 C CNN
 F 1 "GND" H 5500 4120 30  0001 C CNN
 F 2 "" H 5500 4200 60  0000 C CNN
@@
 $EndComp
 $Comp
-L GND #PWR06
+L GND #PWR05
 U 1 1 564714EA
 P 10200 3550
-F 0 "#PWR06" H 10290 3530 30  0001 C CNN
+F 0 "#PWR05" H 10290 3530 30  0001 C CNN
 F 1 "GND" H 10200 3470 30  0001 C CNN
 F 2 "" H 10200 3550 60  0000 C CNN
@@
 $EndComp
 $Comp
-L GND #PWR07
+L GND #PWR06
 U 1 1 56488406
 P 1500 5550
-F 0 "#PWR07" H 1590 5530 30  0001 C CNN
+F 0 "#PWR06" H 1590 5530 30  0001 C CNN
 F 1 "GND" H 1500 5470 30  0001 C CNN
 F 2 "" H 1500 5550 60  0000 C CNN
@@
 $EndComp
 $Comp
-L +BATT #PWR08
+L +BATT #PWR07
 U 1 1 56488459
 P 2750 5550
-F 0 "#PWR08" H 2750 5510 30  0001 C CNN
+F 0 "#PWR07" H 2750 5510 30  0001 C CNN
 F 1 "+BATT" H 2830 5580 30  0000 C CNN
 F 2 "" H 2750 5550 60  0000 C CNN
@@
 $EndComp
 $Comp
-L +BATT #PWR09
+L +BATT #PWR08
 U 1 1 56488624
 P 5400 3200
-F 0 "#PWR09" H 5400 3160 30  0001 C CNN
+F 0 "#PWR08" H 5400 3160 30  0001 C CNN
 F 1 "+BATT" H 5480 3230 30  0000 C CNN
 F 2 "" H 5400 3200 60  0000 C CNN
@@
 $EndComp
 $Comp
-L +BATT #PWR010
+L +BATT #PWR09
 U 1 1 56488665
 P 6000 3350
-F 0 "#PWR010" H 6000 3310 30  0001 C CNN
+F 0 "#PWR09" H 6000 3310 30  0001 C CNN
 F 1 "+BATT" H 6080 3380 30  0000 C CNN
 F 2 "" H 6000 3350 60  0000 C CNN
@@
 $EndComp
 Wire Wire Line
-	6000 3350 6100 3350
-Wire Wire Line
-	6100 3350 6400 3350
-Wire Wire Line
-	6400 3350 7000 3350
+	6000 3350 7000 3350
 Wire Wire Line
 	6100 3350 6100 3600
@@
 Connection ~ 6400 3350
 Wire Wire Line
-	5400 3200 5500 3200
-Wire Wire Line
-	5500 3200 5800 3200
-Wire Wire Line
-	5800 3200 7000 3200
+	5400 3200 7000 3200
 Wire Wire Line
 	5500 3200 5500 3600
@@
 $EndComp
 $Comp
-L +BATT #PWR012
+L +BATT #PWR010
 U 1 1 56488C25
 P 10650 7550
-F 0 "#PWR012" H 10650 7510 30  0001 C CNN
+F 0 "#PWR010" H 10650 7510 30  0001 C CNN
 F 1 "+BATT" H 10730 7580 30  0000 C CNN
 F 2 "" H 10650 7550 60  0000 C CNN
@@
 	11350 7550 11350 7600
 $Comp
-L GND #PWR013
+L GND #PWR011
 U 1 1 56488E9B
 P 11350 8150
-F 0 "#PWR013" H 11440 8130 30  0001 C CNN
+F 0 "#PWR011" H 11440 8130 30  0001 C CNN
 F 1 "GND" H 11350 8070 30  0001 C CNN
 F 2 "" H 11350 8150 60  0000 C CNN
@@
 $EndComp
 $Comp
-L GND #PWR014
+L GND #PWR012
 U 1 1 56488EC7
 P 11050 8150
-F 0 "#PWR014" H 11140 8130 30  0001 C CNN
+F 0 "#PWR012" H 11140 8130 30  0001 C CNN
 F 1 "GND" H 11050 8070 30  0001 C CNN
 F 2 "" H 11050 8150 60  0000 C CNN
@@
 $EndComp
 $Comp
-L GND #PWR015
+L GND #PWR013
 U 1 1 56489007
 P 11750 9050
-F 0 "#PWR015" H 11840 9030 30  0001 C CNN
+F 0 "#PWR013" H 11840 9030 30  0001 C CNN
 F 1 "GND" H 11750 8970 30  0001 C CNN
 F 2 "" H 11750 9050 60  0000 C CNN
@@
 $EndComp
 $Comp
-L GND #PWR016
+L GND #PWR014
 U 1 1 5648A5B1
 P 2950 9300
-F 0 "#PWR016" H 3040 9280 30  0001 C CNN
+F 0 "#PWR014" H 3040 9280 30  0001 C CNN
 F 1 "GND" H 2950 9220 30  0001 C CNN
 F 2 "" H 2950 9300 60  0000 C CNN
@@
 $EndComp
 Wire Wire Line
-	2950 9150 2950 9200
-Wire Wire Line
-	2950 9200 2950 9300
+	2950 9150 2950 9300
 Wire Wire Line
 	2850 9150 2850 9200
 Wire Wire Line
-	2850 9200 2950 9200
-Wire Wire Line
-	2950 9200 3050 9200
+	2850 9200 3050 9200
 Connection ~ 2950 9200
 Wire Wire Line
 	3050 9200 3050 9150
 $Comp
-L GND #PWR017
+L GND #PWR015
 U 1 1 5648A6B6
 P 4200 8300
-F 0 "#PWR017" H 4290 8280 30  0001 C CNN
+F 0 "#PWR015" H 4290 8280 30  0001 C CNN
 F 1 "GND" H 4200 8220 30  0001 C CNN
 F 2 "" H 4200 8300 60  0000 C CNN
@@
 $EndComp
 Wire Wire Line
-	3950 8700 4100 8700
-Wire Wire Line
-	4100 8700 4200 8700
+	3950 8700 4200 8700
 Wire Wire Line
 	4100 8700 4100 8800
 Wire Wire Line
-	3950 8600 4400 8600
-Wire Wire Line
-	4400 8600 4500 8600
+	3950 8600 4500 8600
 Wire Wire Line
 	4400 8600 4400 8800
@@
 	4700 8450 4700 8800
 $Comp
-L +BATT #PWR018
+L +BATT #PWR016
 U 1 1 5648A8C3
 P 4200 8700
-F 0 "#PWR018" H 4200 8660 30  0001 C CNN
+F 0 "#PWR016" H 4200 8660 30  0001 C CNN
 F 1 "+BATT" H 4280 8730 30  0000 C CNN
 F 2 "" H 4200 8700 60  0000 C CNN
@@
 $EndComp
 $Comp
-L +BATT #PWR019
+L +BATT #PWR017
 U 1 1 5648A8FB
 P 4500 8600
-F 0 "#PWR019" H 4500 8560 30  0001 C CNN
+F 0 "#PWR017" H 4500 8560 30  0001 C CNN
 F 1 "+BATT" H 4580 8630 30  0000 C CNN
 F 2 "" H 4500 8600 60  0000 C CNN
@@
 Connection ~ 4400 8600
 $Comp
-L GND #PWR020
+L GND #PWR018
 U 1 1 5648A9D2
 P 4100 9350
-F 0 "#PWR020" H 4190 9330 30  0001 C CNN
+F 0 "#PWR018" H 4190 9330 30  0001 C CNN
 F 1 "GND" H 4100 9270 30  0001 C CNN
 F 2 "" H 4100 9350 60  0000 C CNN
@@
 $EndComp
 $Comp
-L GND #PWR021
+L GND #PWR019
 U 1 1 5648AA0A
 P 4400 9350
-F 0 "#PWR021" H 4490 9330 30  0001 C CNN
+F 0 "#PWR019" H 4490 9330 30  0001 C CNN
 F 1 "GND" H 4400 9270 30  0001 C CNN
 F 2 "" H 4400 9350 60  0000 C CNN
@@
 $EndComp
 $Comp
-L GND #PWR022
+L GND #PWR020
 U 1 1 5648AA42
 P 4700 9350
-F 0 "#PWR022" H 4790 9330 30  0001 C CNN
+F 0 "#PWR020" H 4790 9330 30  0001 C CNN
 F 1 "GND" H 4700 9270 30  0001 C CNN
 F 2 "" H 4700 9350 60  0000 C CNN
@@
 $EndComp
 $Comp
-L +BATT #PWR023
+L +BATT #PWR021
 U 1 1 5648AF51
 P 5500 8500
-F 0 "#PWR023" H 5500 8460 30  0001 C CNN
+F 0 "#PWR021" H 5500 8460 30  0001 C CNN
 F 1 "+BATT" H 5580 8530 30  0000 C CNN
 F 2 "" H 5500 8500 60  0000 C CNN
@@
 	5500 8500 5650 8500
 Wire Wire Line
-	5650 8400 5650 8500
-Wire Wire Line
-	5650 8500 5650 8600
+	5650 8400 5650 8600
 Connection ~ 5650 8500
 Text Label 6550 8600 2    60   ~ 0
@@
 P 6550 2150
 F 0 "R3" V 6630 2000 50  0000 C CNN
-F 1 "51R" V 6550 2150 50  0000 C CNN
+F 1 "100R" V 6550 2150 50  0000 C CNN
 F 2 "Resistors:RES_0402" V 6630 2250 28  0001 C CNN
 F 3 "" H 6550 2150 60  0000 C CNN
@@
 $EndComp
 $Comp
-L GND #PWR024
+L GND #PWR022
 U 1 1 5648A1C4
 P 5450 2350
-F 0 "#PWR024" H 5540 2330 30  0001 C CNN
+F 0 "#PWR022" H 5540 2330 30  0001 C CNN
 F 1 "GND" H 5450 2270 30  0001 C CNN
 F 2 "" H 5450 2350 60  0000 C CNN
@@
 P 10850 2600
 F 0 "R5" V 10750 2600 50  0000 C CNN
-F 1 "51R" V 10850 2600 50  0000 C CNN
+F 1 "100R" V 10850 2600 50  0000 C CNN
 F 2 "Resistors:RES_0402" V 10930 2700 28  0001 C CNN
 F 3 "" H 10850 2600 60  0000 C CNN
@@
 P 10850 2900
 F 0 "R6" V 10950 2850 50  0000 C CNN
-F 1 "51R" V 10850 2900 50  0000 C CNN
+F 1 "100R" V 10850 2900 50  0000 C CNN
 F 2 "Resistors:RES_0402" V 10930 3000 28  0001 C CNN
 F 3 "" H 10850 2900 60  0000 C CNN
@@
 	11100 2900 11250 2900
 $Comp
-L GND #PWR025
+L GND #PWR023
 U 1 1 5648A87D
 P 11900 2600
-F 0 "#PWR025" H 11990 2580 30  0001 C CNN
+F 0 "#PWR023" H 11990 2580 30  0001 C CNN
 F 1 "GND" H 11900 2520 30  0001 C CNN
 F 2 "" H 11900 2600 60  0000 C CNN
@@
 $EndComp
 $Comp
-L GND #PWR026
+L GND #PWR024
 U 1 1 5648A8C5
 P 11900 2900
-F 0 "#PWR026" H 11990 2880 30  0001 C CNN
+F 0 "#PWR024" H 11990 2880 30  0001 C CNN
 F 1 "GND" H 11900 2820 30  0001 C CNN
 F 2 "" H 11900 2900 60  0000 C CNN
@@
 	10750 8650 10450 8650
 Wire Wire Line
-	10650 7550 11050 7550
-Wire Wire Line
-	11050 7550 11350 7550
-Wire Wire Line
-	11350 7550 11750 7550
-Wire Wire Line
-	11750 7550 12050 7550
+	10650 7550 12050 7550
 Wire Wire Line
 	12050 7550 12050 8150
@@
 	12050 8350 11750 8350
 Wire Wire Line
-	11750 8000 11750 8350
-Wire Wire Line
-	11750 8350 11750 8450
+	11750 8000 11750 8450
 Connection ~ 11750 8350
 $Comp
@@
 $EndComp
 $Comp
-L +BATT #PWR027
+L +BATT #PWR025
 U 1 1 5648BB9C
 P 2600 2350
-F 0 "#PWR027" H 2600 2310 30  0001 C CNN
+F 0 "#PWR025" H 2600 2310 30  0001 C CNN
 F 1 "+BATT" H 2680 2380 30  0000 C CNN
 F 2 "" H 2600 2350 60  0000 C CNN
@@
 	2400 2350 2600 2350
 $Comp
-L GND #PWR028
+L GND #PWR026
 U 1 1 5648BD96
 P 2500 2550
-F 0 "#PWR028" H 2590 2530 30  0001 C CNN
+F 0 "#PWR026" H 2590 2530 30  0001 C CNN
 F 1 "GND" H 2500 2470 30  0001 C CNN
 F 2 "" H 2500 2550 60  0000 C CNN
@@
 UART_RX
 $Comp
-L GND #PWR029
+L GND #PWR027
 U 1 1 5648CA97
 P 2400 4100
-F 0 "#PWR029" H 2490 4080 30  0001 C CNN
+F 0 "#PWR027" H 2490 4080 30  0001 C CNN
 F 1 "GND" H 2400 4020 30  0001 C CNN
 F 2 "" H 2400 4100 60  0000 C CNN
@@
 Vibro_out
 $Comp
-L STM32F042F6P6 DD?
+L STM32F042F6P6 DD2
 U 1 1 564DD21B
 P 8550 2750
-F 0 "DD?" H 8050 3600 60  0000 C CNN
+F 0 "DD2" H 8050 3600 60  0000 C CNN
 F 1 "STM32F042F6P6" H 8600 3600 60  0000 C CNN
-F 2 "" H 8600 1850 60  0000 C CNN
+F 2 "SO_DIL_TSSOP:TSSOP20" H 8600 1850 60  0001 C CNN
 F 3 "" H 8600 1850 60  0000 C CNN
 	1    8550 2750
