File: CalmaAcc_hw/CalmaAcc.kicad_pcb (KiCad board)
At the start: 2 copper layers, 27 x 17 mm, 27 parts, among them Q1 MMBT2222

Commit message: + gerber
Parts:
- moved XL3 21.6 mm to (133.1, 80.8), turned to 270 degrees
- moved D3 20.2 mm to (149.7, 80.1), turned to 180 degrees
- moved R5 19.8 mm to (148.9, 81.9), turned to 180 degrees
- moved DD2 17.9 mm to (140.8, 88.5), turned to 180 degrees
- moved D1 17.3 mm to (140.8, 95.1)
- moved D4 17.3 mm to (129.5, 80.2)
- moved C10 17.1 mm to (137.4, 81.7), turned to 270 degrees
- moved C9 16.1 mm to (139.7, 81.7), turned to 270 degrees
- moved R6 14.6 mm to (129.2, 82.0)
- moved R3 14.4 mm to (141.2, 93.2), turned to 180 degrees
- moved C4 10.8 mm to (145.0, 89.3), turned to 0 degrees
- moved C5 10.8 mm to (145.0, 87.8), turned to 0 degrees
- moved C8 8.46 mm to (136.6, 89.2), turned to 180 degrees
- moved C6 8.11 mm to (136.5, 86.2), turned to 180 degrees
- moved C7 7.69 mm to (136.5, 87.7), turned to 180 degrees
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Routing:
- net GND: track 0.00 -> 121.2 mm, vias 0 -> 20
- net +BATT: track 0.00 -> 84.4 mm, vias 0 -> 5
- net /I2C_SCL: track 0.00 -> 13.8 mm, vias 0 -> 2
- net /UART_RX: track 0.00 -> 13.7 mm
- net /ACC_INT1: track 0.00 -> 13.7 mm, vias 0 -> 2
- net /I2C_SDA: track 0.00 -> 13.0 mm, vias 0 -> 2
- net Net-(DD2-Pad13): track 0.00 -> 11.8 mm
- net /UART_TX: track 0.00 -> 11.6 mm
- net Net-(DD2-Pad14): track 0.00 -> 10.5 mm, vias 0 -> 2
- net Net-(DD2-Pad12): track 0.00 -> 9.73 mm, vias 0 -> 2
- net /Vibro_out: track 0.00 -> 9.57 mm
- net /SWCLK: track 0.00 -> 8.84 mm
- net /SWDIO: track 0.00 -> 5.19 mm, vias 0 -> 1
- net Net-(C3-Pad1): track 0.00 -> 2.44 mm
- net Net-(D3-PadA): track 0.00 -> 2.11 mm
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- added copper zone on B.Cu, net GND
- added copper zone on F.Cu, net GND
Other:
- rule pad_to_mask_clearance: 0.2 -> 0.1

Commit message: + TSSOP20
Parts:
- removed C8: 0.1u, Capacitors:CAP_0402
- DD2: value STM32F042G4 -> STM32F042F6P6; footprint QFN_DFN:UFQFPN28 -> SO_DIL_TSSOP:TSSOP20
- R3, R5, R6: value 51R -> 100R
Connections:
- DD2 pad 1: Net-(DD2-Pad1) -> (no net)
- DD2 pad 15: Net-(DD2-Pad15) -> GND
- DD2 pad 16: GND -> +BATT
- DD2 pad 17: +BATT -> (no net)
- DD2 pad 18: +BATT -> (no net)
- DD2 pad 19: (no net) -> /SWDIO
- DD2 pad 2: (no net) -> /I2C_SDA
- DD2 pad 20: (no net) -> /SWCLK
- DD2 pad 3: (no net) -> /I2C_SCL
- DD2 pad 7: Net-(DD2-Pad7) -> (no net)
Routing:
- net Net-(DD2-Pad14): track 10.5 -> 0.42 mm, vias 2 -> 0
- net +BATT: track 84.4 -> 94.1 mm, vias 5 -> 6
- net /I2C_SDA: track 13.0 -> 4.52 mm, vias 2 -> 1
- net /SWCLK: track 8.84 -> 2.35 mm
- net /ACC_INT1: track 13.7 -> 17.7 mm, vias 2 -> 3
- net Net-(DD2-Pad13): track 11.8 -> 15.9 mm, vias 0 -> 1
- net /UART_RX: track 13.7 -> 16.6 mm, vias 0 -> 1
- net /SWDIO: track 5.19 -> 7.64 mm, vias 1 -> 2
- net Net-(DD2-Pad12): track 9.73 -> 12.1 mm, vias 2 -> 1
- net /I2C_SCL: track 13.8 -> 13.3 mm, vias 2 -> 1
- removed copper zone on B.Cu, net GND
- removed copper zone on F.Cu, net GND

Commit message: +gerber
Parts:
- moved XL1 20.0 mm to (149.5, 94.7), turned to 180 degrees
- moved D3 18.9 mm to (138.1, 95.1), turned to 0 degrees
- moved D1 17.2 mm to (149.5, 80.2)
- moved R5 15.9 mm to (137.8, 93.3), turned to 0 degrees
- moved XL4 15.1 mm to (129.8, 94.7)
- moved R3 13.5 mm to (148.8, 82.1), turned to 0 degrees
- moved C7 10.5 mm to (147.0, 87.9), turned to 0 degrees
- moved C6 10.5 mm to (147.0, 86.4), turned to 0 degrees
- moved C4 9.21 mm to (135.8, 89.2), turned to 180 degrees
- moved C5 9.16 mm to (135.8, 87.7), turned to 180 degrees
- moved R4 4.38 mm to (146.2, 82.9), turned to 270 degrees
- moved R2 1.74 mm to (133.5, 89.2)
- moved DD2 0.70 mm to (141.3, 88.0), turned to 270 degrees
Routing:
- net GND: track 121.2 -> 148.9 mm, vias 20 -> 26
- net +BATT: track 94.1 -> 77.0 mm, vias 6 -> 3
- net /SWCLK: track 2.35 -> 13.8 mm
- net Net-(DD2-Pad14): track 0.42 -> 11.2 mm
- net /UART_RX: track 16.6 -> 5.91 mm, vias 1 -> 0
- net /Vibro: track 2.02 -> 11.9 mm
- net /SWDIO: track 7.64 -> 15.6 mm, vias 2 -> 0
- net Net-(DD2-Pad12): track 12.1 -> 6.70 mm, vias 1 -> 0
- net /ACC_INT1: track 17.7 -> 12.7 mm, vias 3 -> 2
- net /I2C_SDA: track 4.52 -> 8.19 mm, vias 1 -> 0
- net /UART_TX: track 11.6 -> 8.04 mm
- net /I2C_SCL: track 13.3 -> 11.5 mm, vias 1 -> 2
- net Net-(DD2-Pad13): track 15.9 -> 17.4 mm, vias 1 -> 2
- net /Vibro_out: track 9.57 -> 10.2 mm
- net Net-(Q1-Pad1): track 2.06 -> 2.60 mm
- added copper zone on B.Cu, net GND
- added copper zone on F.Cu, net GND
